File: optical6dof-evaluationboard/Optical.kicad_pcb (KiCad board)
At the start: 4 copper layers, 20.2 x 12 mm, 29 parts, among them Q1 BPW40, Q2 BPW40, Q3 BPW40, Q4 BPW40, Q5 BPW40, Q6 BPW40, U1 AD7689BCBZ-RL7

Commit message: new pcb
Parts:
- removed ? (x5): , 
- added C6: 10uF, Capacitor_SMD:C_0402_1005Metric, B.Cu at (175.0, 72.3)
- added C7: 10uF, Capacitor_SMD:C_0402_1005Metric, F.Cu at (157.0, 58.6)
- added C8: 100uF, Capacitor_SMD:C_0402_1005Metric, B.Cu at (172.5, 74.1)
- added C9: 10uF, Capacitor_SMD:C_0402_1005Metric, B.Cu at (173.5, 75.1)
- added J1: FFC2B28-12-G, library:GCT_FFC2B28-12-G, B.Cu at (176.3, 77.3)
- added R10: 220r, library:0402, F.Cu at (161.3, 59.5)
- C1: value 100nF -> 100uF
- C2: value 100uF -> 1uF; moved to B.Cu
- C3: value 10uF -> 4.7nF; moved to B.Cu
- C4: value 0.1uF -> 1uF; moved to B.Cu
- C5: value 10uF -> 100uF; moved to B.Cu
- D1, D2, D3: footprint LED_SMD:LED_0402_1005Metric -> library:APDA3020P3C-P22
- Q1, Q2, Q3, Q4, Q5, Q6: value BPW40 -> APDA3020P3C-P22; footprint library:sidewaysled -> library:APDA3020P3C-P22
- R1, R2, R4, R5, R6: value 24.7k -> 2.2K; footprint Resistor_SMD:R_0201_0603Metric -> library:0402
- R3: value 24.7k -> 2.2K; moved to B.Cu
- R7: value 200r -> 2.2K; footprint Resistor_SMD:R_0201_0603Metric -> library:0402
- R8, R9: value 200r -> 220r; footprint Resistor_SMD:R_0201_0603Metric -> library:0402
- U1: value AD7689BCBZ-RL7 -> ADS1262IPWR; footprint library:CB_20_12_ADI -> library:SOP65P640X120-28N; moved to B.Cu
- moved Q4 72.1 mm to (148.1, 32.6), turned to -150 degrees
- moved Q3 68.2 mm to (139.4, 37.6), turned to -150 degrees
- moved R4 68.2 mm to (139.4, 35.6), turned to -150 degrees
- moved R5 64.6 mm to (148.1, 30.6), turned to -150 degrees
- moved R6 56.7 mm to (185.2, 54.0), turned to 90 degrees
- moved Q5 52.7 mm to (183.5, 53.0), turned to 90 degrees
- moved R7 48.8 mm to (185.2, 64.0)
- moved D2 48.6 mm to (153.8, 52.4), turned to 30 degrees
- moved R9 47.8 mm to (156.1, 53.5), turned to -60 degrees
- moved Q6 46.1 mm to (183.5, 63.0), turned to 90 degrees
- moved D3 43.5 mm to (163.5, 58.0), turned to -90 degrees
- moved R8 40.4 mm to (153.6, 61.0), turned to 60 degrees
- moved C1 40.1 mm to (157.0, 57.4), turned to 0 degrees
- moved D1 36.2 mm to (153.8, 63.6), turned to 150 degrees
- moved C5 31.4 mm to (176.0, 73.3), turned to -135 degrees
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Connections:
- C2 pad 2: VDD -> Net-(U1-BYPASS)
- C3 pad 1: GND -> Net-(U1-CAPP)
- C3 pad 2: VDD -> Net-(U1-CAPN)
- C4 pad 2: VDD -> Net-(U1-REFOUT)
- C5 pad 2: Net-(U1-WREF) -> VDD
- Q1 pad 1: /A1 -> VDD
- Q1 pad 2: VDD -> /A1
- Q3 pad 1: /B1 -> VDD
- Q3 pad 2: VDD -> /B1
- Q5 pad 1: /C1 -> VDD
- Q5 pad 2: VDD -> /C1
- R3 pad 1: /B1 -> START
- R3 pad 2: GND -> VDD_digital
- R4 pad 1: /B2 -> /B1
- R5 pad 1: /C1 -> /B2
- R6 pad 1: /C2 -> /C1
- R7 pad 1: Net-(D1-K) -> /C2
- R8 pad 1: Net-(D2-K) -> Net-(D1-K)
- R9 pad 1: Net-(D3-K) -> Net-(D2-K)
Routing:
- net /C2: track 0.00 -> 75.3 mm, vias 0 -> 2
- net /C1: track 1.42 -> 67.8 mm, vias 0 -> 2
- net VDD_digital: track 0.00 -> 21.8 mm
- net GND: track 4.54 -> 19.8 mm, vias 5 -> 142
- net START: track 0.00 -> 13.2 mm
- net /B2: track 1.13 -> 13.6 mm, vias 0 -> 2
- net CS: track 0.00 -> 10.5 mm
- net /SCK: track 9.08 -> 0.00 mm
- net VDD: track 14.1 -> 5.26 mm, vias 6 -> 12
- net /SDO: track 8.03 -> 0.00 mm, vias 1 -> 0
- net SCLK: track 0.00 -> 7.82 mm
- net MOSI: track 0.00 -> 6.82 mm
- net MISO: track 0.00 -> 5.76 mm
- net /B1: track 0.00 -> 5.04 mm, vias 0 -> 2
- net /CNV: track 4.85 -> 0.00 mm
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- added copper zone on In2.Cu, net GND
- added copper zone on B.Cu, net VDD
- added copper zone on B.Cu, net VDD_digital
- removed copper zone on F.Cu, net GND
- removed copper zone on In1.Cu, net VDD
- removed copper zone on In2.Cu, net VDD
Other:
- board size 20.2 x 12 mm -> 60 x 60 mm
- board text added: "SoftCON"
- board text added: "Softcon"
