File: optical6dof-evaluationboard/Optical.kicad_sch (KiCad schematic)
At the start: 23 parts, among them U1 MAX11617EWE+T

Commit message: changes
Parts:
- removed Q1, Q2, Q3: ~, library:0603_sidemount, symbol library:dual_phototransistor
- removed U1: MAX11617EWE+T, library:21-0491G_W162E2-1_MXM, symbol MAX11617EWE:MAX11617EWE+T
- added C1: 100nF, Capacitor_SMD:C_0402_1005Metric, symbol Device:C
- added C2: 100uF, Capacitor_SMD:C_0402_1005Metric, symbol Device:C
- added C3, C5: 10uF, Capacitor_SMD:C_0402_1005Metric, symbol Device:C
- added C4: 0.1uF, Capacitor_SMD:C_0402_1005Metric, symbol Device:C
- added Q1, Q2, Q3, Q4, Q5, Q6: BPW40, library:sidewaysled, symbol Sensor_Optical:BPW40
- R1, R2, R3, R4, R5, R6: value 1.5k -> 24.7k; footprint Resistor_SMD:R_01005_0402Metric -> Resistor_SMD:R_0201_0603Metric
- R7, R8, R9: footprint Resistor_SMD:R_01005_0402Metric -> Resistor_SMD:R_0201_0603Metric
- gave numbers to parts that had none: 1
Connections:
- net A1: now also Q1.1 (C)
- net A2: now also Q2.2 (E)
- net B1: now also Q3.1 (C)
- net B2: now also Q4.2 (E)
- net C1: now also Q5.1 (C)
- net C2: now also Q6.2 (E)
- net GND: now also U1.D6 (GND), U1.D8 (GND), U1.E1 (COM), C1.1, C2.1, C3.1, C4.1, C5.1
- net VDD: now also U1.A1 (VIO), U1.B6 (VDD), U1.B8 (VDD), U1.C7 (REFIN), C1.2, C2.2, C3.2, C4.2, Q1.2 (E), Q2.1 (C), Q3.2 (E), Q4.1 (C), Q5.2 (E), Q6.1 (C)
- net 0: now reaches U1.A3 (IN0)
- net 2: now reaches U1.A5 (IN2)
- net 3: now reaches U1.A7 (IN3)
- net SDO: now reaches U1.B2 (SDO)
- net 1: now reaches U1.B4 (IN1)
- net SCK: now reaches U1.C3 (SCK)
- net DIN: now reaches U1.C5 (DIN)
- net at U1.C9 (WREF): now also C5.2
- net CNV: now reaches U1.D2 (CNV)
- net 7: now reaches U1.D4 (IN7)
- net 6: now reaches U1.E3 (IN6)
- net 5: now reaches U1.E5 (IN5)
- net 4: now reaches U1.E7 (IN4)
Other:
- moved on the sheet: D1, D2, D3, R2, R4, R7, R8, R9, TP2, TP4, U1

Commit message: new pcb
Parts:
- removed R7: 200r, Resistor_SMD:R_0201_0603Metric, symbol Device:R
- removed U1: AD7689BCBZ-RL7, library:CB_20_12_ADI, symbol AD7689:AD7689BCBZ-RL7
- added C6, C7, C9: 10uF, Capacitor_SMD:C_0402_1005Metric, symbol Device:C
- added C8: 100uF, Capacitor_SMD:C_0402_1005Metric, symbol Device:C
- added J1: FFC2B28-12-G, library:GCT_FFC2B28-12-G, symbol FFC2B28-12-G:FFC2B28-12-G
- added R10: 220r, library:0402, symbol Device:R
- added R3: 2.2K, Resistor_SMD:R_0201_0603Metric, symbol Device:R
- added U1: ADS1262IPWR, library:SOP65P640X120-28N, symbol ADS1262IPWR:ADS1262IPWR
- C1: value 100nF -> 100uF
- C2: value 100uF -> 1uF
- C3: value 10uF -> 4.7nF
- C4: value 0.1uF -> 1uF
- C5: value 10uF -> 100uF
- D1, D2, D3: footprint LED_SMD:LED_0402_1005Metric -> library:APDA3020P3C-P22; Digikey https://www.digikey.com/en/products/detail/inolux/IN-S42CTQ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 -> https://www.digikey.com/en/products/detail/kingbright/APDA3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
- Q1, Q2, Q3, Q4, Q5, Q6: value BPW40 -> APDA3020P3C-P22; footprint library:sidewaysled -> library:APDA3020P3C-P22; Digikey (none) -> https://www.digikey.com/en/products/detail/kingbright/APDA3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
- R1, R2: value 24.7k -> 2.2K; footprint Resistor_SMD:R_0201_0603Metric -> library:0402; Digikey https://www.digikey.com/en/products/detail/delta-electronic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 -> https://www.digikey.com/en/products/detail/panasonic-indust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
- R4: renamed from R3; value 24.7k -> 2.2K; footprint Resistor_SMD:R_0201_0603Metric -> library:0402; Digikey https://www.digikey.com/en/products/detail/delta-electronic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 -> https://www.digikey.com/en/products/detail/panasonic-indust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
- R5: renamed from R4; value 24.7k -> 2.2K; footprint Resistor_SMD:R_0201_0603Metric -> library:0402; Digikey https://www.digikey.com/en/products/detail/delta-electronic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 -> https://www.digikey.com/en/products/detail/panasonic-indust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
- R6: renamed from R5; value 24.7k -> 2.2K; footprint Resistor_SMD:R_0201_0603Metric -> library:0402; Digikey https://www.digikey.com/en/products/detail/delta-electronic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 -> https://www.digikey.com/en/products/detail/panasonic-indust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
- R7: renamed from R6; value 24.7k -> 2.2K; footprint Resistor_SMD:R_0201_0603Metric -> library:0402; Digikey https://www.digikey.com/en/products/detail/delta-electronic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 -> https://www.digikey.com/en/products/detail/panasonic-indust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
- R8, R9: value 200r -> 220r; footprint Resistor_SMD:R_0201_0603Metric -> library:0402; Digikey https://www.digikey.com/en/products/detail/yageo/RC0100FR-0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 -> https://www.digikey.com/en/products/detail/stackpole-electr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
Connections:
- net A1: now also Q1.2 (E), U1.26 (AIN5); no longer Q1.1 (C)
- net A2: now also U1.25 (AIN4)
- net B1: now also Q3.2 (E), U1.27 (AIN6); no longer Q3.1 (C)
- net B2: now also U1.24 (AIN3)
- net C1: now also Q5.2 (E), U1.23 (AIN2); no longer Q5.1 (C)
- net C2: now also U1.22 (AIN1)
- net GND: now also C6.1, C7.1, C8.1, C9.1, J1.1, J1.4, J1.5, R10.2, U1.15 (XTAL1/CLKIN), U1.18 (DGND), U1.3 (AINCOM), U1.7 (AVSS); no longer C3.1
- net VDD: now also C5.2, Q1.1 (C), Q3.1 (C), Q5.1 (C), C6.2, C7.2, J1.2, J1.3, U1.6 (AVDD); no longer C2.2, C3.2, C4.2, Q1.2 (E), Q3.2 (E), Q5.2 (E)
- net at R9.1: now also D2.1 (K); no longer D3.1 (K)
- net at R8.1: now also D1.1 (K); no longer D2.1 (K)
- new net: C3.1, U1.4 (CAPP)
- new net: C3.2, U1.5 (CAPN)
- new net: C2.2, U1.17 (BYPASS)
- new net: C4.2, U1.8 (REFOUT)
- new net: D3.1 (K), R10.1
- new net CS: J1.8, U1.10 (CS)
- new net DataReady: J1.12, U1.14 (DRDY)
- new net MISO: J1.11, U1.13 (DOUT/DRDY)
- new net MOSI: J1.10, U1.12 (DIN)
- new net SCLK: J1.9, U1.11 (SCLK)
- new net START: J1.7, R3.1, U1.9 (START)
- new net VDD_digital: C8.2, C9.2, J1.6, R3.2, U1.19 (DVDD), U1.20 (RESET/PWDN)
- no-connect marks 0 -> 3
Other:
- note added: "ADS1262IPWR"
- note added: "https://www.digikey.com/en/products/detail/everlight-electronics-co-ltd/PT928-6B-F/2675658"
- note added: "https://www.digikey.com/en/products/detail/gct/FFC2B28-12-G/10656933"
- note added: "https://www.digikey.com/en/products/detail/kingbright/APDA3020F3C-P22/16639771"
- note added: "https://www.digikey.com/en/products/detail/kingbright/APDA3020P3C-P22/16639769"
- note added: "phototransistor: https://www.digikey.com/en/products/detail/kingbright/WP3DP3BT-BD-P22/8591564 ir led: https://www.digikey.com/en/products/detail/vishay-semiconductor-opto-division/TSAL4400/1681336"
- note removed: "3.3v/2.42mA"
- note removed: "Ic(on) = 2.42mA max"
- moved on the sheet: R1, R2, R4, R5, R6, R7, TP1, TP2, TP3, TP4, TP5, TP6
